Commit message: refactor: update robot name to 'rove_standard' and add new camera links in URDF

File: src/media/rove_urdf/rove.urdf (robot description, URDF)
Before this commit: robot rove_cursed_aaaah_goofy_design, 39 links, 38 joints
Links:
- removed link vn300_vectornav_pivot
- added link chinese_camera_4; collision mesh filename=meshes/chinese_camera_4.glb; visual mesh filename=meshes/chinese_camera_4.glb
- added link chinese_camera_4_pivot
- added link chinese_camera_5; collision mesh filename=meshes/chinese_camera_5.glb; visual mesh filename=meshes/chinese_camera_5.glb
- added link chinese_camera_5_pivot
- added link chinese_camera_6; collision mesh filename=meshes/chinese_camera_6.glb; visual mesh filename=meshes/chinese_camera_6.glb
- added link chinese_camera_6_pivot
- added link chinese_camera_7; collision mesh filename=meshes/chinese_camera_7.glb; visual mesh filename=meshes/chinese_camera_7.glb
- added link chinese_camera_7_pivot
- added link dji_mid360_2; collision mesh filename=meshes/dji_mid360.glb; visual mesh filename=meshes/dji_mid360.glb
- added link dji_mid360_2_pivot
- added link pole; collision mesh filename=meshes/pole.glb; visual mesh filename=meshes/pole.glb
- added link pole_pivot
- link chinese_camera: geometry collision mesh filename=meshes/chinese_camera.glb; visual mesh filename=meshes/chinese_camera.glb
- link chinese_camera_2: geometry collision mesh filename=meshes/chinese_camera_2.glb; visual mesh filename=meshes/chinese_camera_2.glb
- link chinese_camera_3: geometry collision mesh filename=meshes/chinese_camera_3.glb; visual mesh filename=meshes/chinese_camera_3.glb
Joints:
- removed joint joint_fixed
- removed joint joint_fixed_2
- removed joint joint_fixed_2_offset
- removed joint joint_fixed_offset
- added joint joint_revolute_18: type revolute, parent JointB, child JointGripper_pivot, origin xyz=-1.1728 0.20415 0.378 rpy=0 0 0, axis -1 0 0, limit lower=-3.14159 upper=3.14159 effort=10 velocity=1
- added joint joint_revolute_18_offset: type fixed, parent JointGripper_pivot, child JointGripper, origin xyz=1.1728 -0.20415 -0.378 rpy=0 0 0
- added joint joint_revolute_19: type fixed, parent pole, child chinese_camera_2_pivot, origin xyz=0.024 0.0730961 0.586861 rpy=0 0 0, axis 0 0.23939 0.970923, limit lower=-3.14159 upper=3.14159 effort=10 velocity=1
- added joint joint_revolute_19_offset: type fixed, parent chinese_camera_2_pivot, child chinese_camera_2, origin xyz=-0.0239323 0.014361 -0.00867528 rpy=-1.5708 -1.38778e-16 3.14159
- added joint joint_revolute_20: type fixed, parent pole, child chinese_camera_3_pivot, origin xyz=-0.0730961 0.024 0.586861 rpy=0 0 0, axis 0 -1 0, limit lower=-3.14159 upper=3.14159 effort=10 velocity=1
- added joint joint_revolute_20_offset: type fixed, parent chinese_camera_3_pivot, child chinese_camera_3, origin xyz=-0.0149206 -0.0234735 -0.00886397 rpy=-1.5708 5.55112e-17 -1.5708
- added joint joint_revolute_21: type revolute, parent pole, child chinese_camera_4_pivot, origin xyz=-0.024 -0.0727157 0.587006 rpy=0 0 0, axis 0 -0.46469 0.885474, limit lower=-3.14159 upper=3.14159 effort=10 velocity=1
- added joint joint_revolute_21_offset: type fixed, parent chinese_camera_4_pivot, child chinese_camera_4, origin xyz=0.0248549 -0.0148706 -0.0090392 rpy=-1.5708 -2.22045e-16 1.60237e-31
- added joint joint_revolute_22: type fixed, parent Core, child chinese_camera_5_pivot, origin xyz=-0.447106 0.216081 0.168303 rpy=0 0 0, axis -0.999548 0.0300528 0, limit lower=-3.14159 upper=3.14159 effort=10 velocity=1
- added joint joint_revolute_22_offset: type fixed, parent chinese_camera_5_pivot, child chinese_camera_5, origin xyz=-0.0228113 -0.00141777 -0.0192583 rpy=-1.5708 -5.55112e-17 -1.5708
- added joint joint_revolute_23: type fixed, parent Core, child chinese_camera_6_pivot, origin xyz=0.31746 0.209 0.192576 rpy=0 0 0, axis 1 0 0, limit lower=-3.14159 upper=3.14159 effort=10 velocity=1
- added joint joint_revolute_23_offset: type fixed, parent chinese_camera_6_pivot, child chinese_camera_6, origin xyz=0.031733 -0.000947911 -0.0166233 rpy=-1.5708 5.55112e-17 1.5708
- added joint joint_revolute_24: type fixed, parent JointGripper, child chinese_camera_7_pivot, origin xyz=-1.1936 0.205 0.4155 rpy=0 0 0, axis 0 -0.111961 0.993713, limit lower=-3.14159 upper=3.14159 effort=10 velocity=1
- added joint joint_revolute_24_offset: type fixed, parent chinese_camera_7_pivot, child chinese_camera_7, origin xyz=0.00311921 6.66671e-05 0.0217355 rpy=-1.5708 -5.55112e-17 -1.5708
- joint joint_revolute_10: axis 0 1 0 -> 0 0 1; child ASection_pivot -> dji_mid360_pivot; limit lower=-0.5 upper=3.6 effort=10 velocity=1 -> lower=-3.14159 upper=3.14159 effort=10 velocity=1; origin xyz=-0.4 0.27 0.388 rpy=0 0 0 -> xyz=-9.31322e-11 -2.66092e-11 0.587 rpy=0 0 0; parent Base -> pole; type revolute -> fixed
- joint joint_revolute_10_offset: child ASection -> dji_mid360; origin xyz=0.4 -0.27 -0.388 rpy=0 0 0 -> xyz=0.00112693 0.0015559 0.0289736 rpy=1.5708 0 1.5708; parent ASection_pivot -> dji_mid360_pivot
- joint joint_revolute_11: axis 0 -1 0 -> 0 0 -1; child JointA_pivot -> dji_mid360_2_pivot; origin xyz=-0.7 0.255 0.378 rpy=0 0 0 -> xyz=4.59098e-18 0 0.574 rpy=0 0 0; parent ASection -> pole; type revolute -> fixed
- joint joint_revolute_11_offset: child JointA -> dji_mid360_2; origin xyz=0.7 -0.255 -0.378 rpy=0 0 0 -> xyz=0.000551953 -0.000521468 -0.0284671 rpy=-1.5708 0 1.5708; parent JointA_pivot -> dji_mid360_2_pivot
- joint joint_revolute_12: axis -1 0 0 -> 0 1 0; child BSection_pivot -> chinese_camera_pivot; origin xyz=-0.767647 0.205 0.378 rpy=0 0 0 -> xyz=0.0725343 -0.024 0.587101 rpy=0 0 0; parent JointA -> pole; type revolute -> fixed
- joint joint_revolute_12_offset: child BSection -> chinese_camera; origin xyz=0.767647 -0.205 -0.378 rpy=0 0 0 -> xyz=0.0154955 0.0243019 -0.00922952 rpy=-1.5708 0 1.5708; parent BSection_pivot -> chinese_camera_pivot
- joint joint_revolute_13: axis 0 1 0 -> 0 0 1; child JointB_pivot -> Base_pivot; limit lower=-1.6 upper=1.6 effort=10 velocity=1 -> lower=-3.14159 upper=3.14159 effort=10 velocity=1; origin xyz=-1.1 0.205 0.378 rpy=0 0 0 -> xyz=-0.399414 0.209923 0.221123 rpy=0 0 0; parent BSection -> Core
- joint joint_revolute_13_offset: child JointB -> Base; origin xyz=1.08936 -0.205 -0.378 rpy=0 0 0 -> xyz=0.399414 -0.209923 -0.15 rpy=0 0 0; parent JointB_pivot -> Base_pivot
- joint joint_revolute_14: axis -1 0 0 -> 0 1 0; child JointGripper_pivot -> ASection_pivot; limit lower=-3.14159 upper=3.14159 effort=10 velocity=1 -> lower=-0.5 upper=3.6 effort=10 velocity=1; origin xyz=-1.1728 0.20415 0.378 rpy=0 0 0 -> xyz=-0.4 0.27 0.388 rpy=0 0 0; parent JointB -> Base
- joint joint_revolute_14_offset: child JointGripper -> ASection; origin xyz=1.1728 -0.20415 -0.378 rpy=0 0 0 -> xyz=0.4 -0.27 -0.388 rpy=0 0 0; parent JointGripper_pivot -> ASection_pivot
- joint joint_revolute_15: axis -0.999548 0.0300528 0 -> 0 -1 0; child chinese_camera_pivot -> JointA_pivot; origin xyz=-0.447106 0.216081 0.168303 rpy=0 0 0 -> xyz=-0.7 0.255 0.378 rpy=0 0 0; parent Core -> ASection; type fixed -> revolute
- joint joint_revolute_15_offset: child chinese_camera -> JointA; origin xyz=-0.0228113 -0.00141777 -0.0192583 rpy=-1.5708 -5.55112e-17 -1.5708 -> xyz=0.7 -0.255 -0.378 rpy=0 0 0; parent chinese_camera_pivot -> JointA_pivot
- joint joint_revolute_16: axis 1 0 0 -> -1 0 0; child chinese_camera_2_pivot -> BSection_pivot; origin xyz=0.31746 0.209 0.192576 rpy=0 0 0 -> xyz=-0.767647 0.205 0.378 rpy=0 0 0; parent Core -> JointA; type fixed -> revolute
- joint joint_revolute_16_offset: child chinese_camera_2 -> BSection; origin xyz=0.031733 -0.000947911 -0.0166233 rpy=-1.5708 5.55112e-17 1.5708 -> xyz=0.767647 -0.205 -0.378 rpy=0 0 0; parent chinese_camera_2_pivot -> BSection_pivot
- joint joint_revolute_17: axis 0 -0.111961 0.993713 -> 0 1 0; child chinese_camera_3_pivot -> JointB_pivot; limit lower=-3.14159 upper=3.14159 effort=10 velocity=1 -> lower=-1.6 upper=1.6 effort=10 velocity=1; origin xyz=-1.1936 0.205 0.4155 rpy=0 0 0 -> xyz=-1.1 0.205 0.378 rpy=0 0 0; parent JointGripper -> BSection; type fixed -> revolute
- joint joint_revolute_17_offset: child chinese_camera_3 -> JointB; origin xyz=0.00311921 6.66671e-05 0.0217355 rpy=-1.5708 -5.55112e-17 -1.5708 -> xyz=1.08936 -0.205 -0.378 rpy=0 0 0; parent chinese_camera_3_pivot -> JointB_pivot
- joint joint_revolute_9: child Base_pivot -> pole_pivot; origin xyz=-0.399414 0.209923 0.221123 rpy=0 0 0 -> xyz=0.31746 0.209 0.221123 rpy=0 0 0; type revolute -> fixed
- joint joint_revolute_9_offset: child Base -> pole; origin xyz=0.399414 -0.209923 -0.221123 rpy=0 0 0 -> xyz=-0.0467844 0.000515604 -0.00281394 rpy=0 0 -1.5708; parent Base_pivot -> pole_pivot
